File: pcb/rode-nt-usb-c.kicad_pcb (KiCad board)
At the start: 2 copper layers, 36 x 15 mm, 6 parts, among them J1 USB_C_Receptacle_USB2.0_16P, J2 Conn_01x05_Pin

Commit message: Update design
Routing:
- net D-: track 35.0 -> 36.7 mm
- net Net-(J1-CC2): track 17.5 -> 16.9 mm
- net Net-(J1-CC1): track 17.5 -> 16.9 mm
